Commit message: LiDAR now seems to make sense. Doesn't get too long range though.

File: ros/src/romipi_florence/urdf/florence_with_lidar.urdf.xacro (robot description, xacro)
@@ -10,5 +10,5 @@
   <!-- LIDAR -->
   <xacro:ld06_lidar_device name="lidar_1" parent="base_link" ros_topic="lidar_1/scan_filtered">
-    <origin xyz="0.360 0 0.181" rpy="3.14 0 0" />
+    <origin xyz="0.360 0 0.181" rpy="0 0 0" />
   </xacro:ld06_lidar_device>
   <!-- Lidar sensors -->
