Commit message: Placed the back caster in the right place

File: ros/src/romipi_description/urdf/romipi.gazebo.xacro (robot description, xacro)
@@ -1,6 +1,6 @@
 <?xml version="1.0"?>
 <robot name="romipi_sim" xmlns:xacro="http://ros.org/wiki/xacro">
-  <xacro:arg name="laser_visual" default="false"/>
-  <xacro:arg name="imu_visual"   default="false"/>
+  <xacro:arg name="laser_visual" default="true"/>
+  <xacro:arg name="imu_visual"   default="true"/>
   <gazebo reference="base_link">
     <material>Gazebo/DarkGrey</material>

File: ros/src/romipi_description/urdf/romipi.urdf.xacro (robot description, xacro)
@@ -90,5 +90,5 @@
     <parent link="base_link"/>
     <child link="caster_back_link"/>
-    <origin xyz="-0.0441 0 0.0" rpy="0 0 0"/>
+    <origin xyz="-0.0441 0.0435 0.0" rpy="0 0 0"/>
   </joint>
   <link name="caster_back_link">

Commit message: Bringing the project in line with my updates to Romipi project.

File: ros/src/romipi_description/urdf/romipi.gazebo.xacro (robot description, xacro)
@@ -1,6 +1,6 @@
 <?xml version="1.0"?>
 <robot name="romipi_sim" xmlns:xacro="http://ros.org/wiki/xacro">
-  <xacro:arg name="laser_visual" default="true"/>
-  <xacro:arg name="imu_visual"   default="true"/>
+  <xacro:arg name="laser_visual" default="false"/>
+  <xacro:arg name="imu_visual"   default="false"/>
   <gazebo reference="base_link">
     <material>Gazebo/DarkGrey</material>
@@ -60,4 +60,7 @@
       <wheelTorque>10</wheelTorque>
       <rosDebugLevel>na</rosDebugLevel>
+      <publishOdomTF>true</publishOdomTF>
+      <odometrySource>world</odometrySource>
+      <odometryRate>20.0</odometryRate>
     </plugin>
   </gazebo>
@@ -90,9 +93,22 @@
     </plugin>
   </gazebo>
-  <gazebo reference="base_scan">
+  <!-- ****** cameras ****** -->
+  <xacro:include filename="simple_camera.urdf.xacro" />
+  <xacro:simple_camera camera_name="camera1" parent_link="base_link" >
+    <origin xyz="0.03 0 0.06" rpy="0 0 0" />
+  </xacro:simple_camera>
+  <!-- ****** LiDAR ****** -->
+  <xacro:include filename="lidar.xacro" />
+  <!-- LIDAR -->
+  <xacro:lidar_device name="base_scan" parent="base_link" ros_topic="base_scan/scan">
+    <origin xyz="0.0 0.0 0.181" rpy="0 0 0" />
+  </xacro:lidar_device>
+  <!-- Lidar sensors -->
+  <gazebo reference="base_scan_link">
     <material>Gazebo/FlatBlack</material>
     <sensor type="ray" name="lds_lfcd_sensor">
       <pose>0 0 0 0 0 0</pose>
       <visualize>$(arg laser_visual)</visualize>
+      <update_rate>40</update_rate>
       <ray>
         <scan>
@@ -116,7 +132,6 @@
       </ray>
       <plugin name="gazebo_ros_lds_lfcd_controller" filename="libgazebo_ros_laser.so">
-        <topicName>scan</topicName>
-        <frameName>base_scan</frameName>
-        <update_rate>1800</update_rate>
+        <topicName>base_scan/scan</topicName>
+        <frameName>base_scan_link</frameName>
       </plugin>
     </sensor>

File: ros/src/romipi_description/urdf/romipi.urdf.xacro (robot description, xacro)
@@ -3,4 +3,15 @@
   <xacro:include filename="$(find romipi_description)/urdf/common_properties.xacro"/>
   <xacro:include filename="$(find romipi_description)/urdf/romipi.gazebo.xacro"/>
+  <xacro:property name="base_link_mass" value="8.2573504e-01" />
+  <xacro:property name="base_link_colision_l" value="0.1635" />
+  <xacro:property name="base_link_colision_w" value="0.145" />
+  <xacro:property name="base_link_colision_h" value="0.05" />
+  <xacro:property name="wheel_mass" value="2.8498940e-02" />
+  <xacro:property name="wheel_width" value="0.018" />
+  <xacro:property name="wheel_radius" value="0.0345" />
+  <xacro:property name="caster_mass" value="0.0005" />
+  <xacro:property name="caster_colision_l" value="0.01" />
+  <xacro:property name="caster_colision_w" value="0.01" />
+  <xacro:property name="caster_colision_h" value="0.01" />
   <link name="base_footprint"/>
   <joint name="base_joint" type="fixed">
@@ -20,13 +31,18 @@
       <origin xyz="0.0 0.0 0.0315" rpy="0 0 0"/>
       <geometry>
-        <box size="0.1635 0.145 0.05"/>
+        <box size="${base_link_colision_l} ${base_link_colision_w} ${base_link_colision_h}"/>
       </geometry>
     </collision>
     <inertial>
-      <origin xyz="0 0 0" rpy="0 0 0"/>
-      <mass value="8.2573504e-01"/>
-      <inertia ixx="2.2124416e-03" ixy="-1.2294101e-05" ixz="3.4938785e-05"
-               iyy="2.1193702e-03" iyz="-5.0120904e-06"
-               izz="2.0064271e-03" />
+      <origin xyz="0 0 0.0315" rpy="0 0 ${pi/2}"/>
+      <mass value="${base_link_mass}" />
+      <!-- According to https://en.wikipedia.org/wiki/List_of_moments_of_inertia#List_of_3D_inertia_tensors
+      We want Ixx = (1/12) * m * (l^2 + h^2) = 0.068811253 * (0.05^2 + 0.1635^2) = 0.002011508 = 2.011508e-03
+              Iyy = (1/12) * m * (w^2 + h^2) = 0.068811253 * (0.145^2 + 0.1635^2) = 0.003286236 = 3.286236e-03
+              Izz = (1/12) * m * (w^2 + l^2) = 0.068811253 * (0.145^2 + 0.05^2) = 0.001618785 = 1.618785e-03
+              -->
+      <inertia ixx="${(1/12) * base_link_mass * (base_link_colision_l**2 + base_link_colision_h**2)}" ixy="0" ixz="0"
+               iyy="${(1/12) * base_link_mass * (base_link_colision_w**2 + base_link_colision_h**2)}" iyz="0"
+               izz="${(1/12) * base_link_mass * (base_link_colision_w**2 + base_link_colision_l**2)}" />
     </inertial>
   </link>
@@ -34,5 +50,5 @@
     <parent link="base_link"/>
     <child link="wheel_left_link"/>
-    <origin xyz="0.0 0.07 0.0345" rpy="0 0 0"/>
+    <origin xyz="0.0 0.07 ${wheel_radius}" rpy="0 0 0"/>
     <axis xyz="0 1 0"/>
   </joint>
@@ -48,13 +64,21 @@
       <origin xyz="0 0 0" rpy="1.57 0 0"/>
       <geometry>
-        <cylinder length="0.018" radius="0.0345"/>
+        <cylinder length="${wheel_width}" radius="${wheel_radius}"/>
       </geometry>
     </collision>
     <inertial>
-      <origin xyz="0 0 0" />
-      <mass value="2.8498940e-02" />
-      <inertia ixx="1.1175580e-05" ixy="-4.2369783e-11" ixz="-5.9381719e-09"
-               iyy="1.1192413e-05" iyz="-1.4400107e-11"
-               izz="2.0712558e-05" />
+      <origin xyz="0 0 0" rpy="1.57 0 0"/>
+      <geometry>
+        <cylinder length="${wheel_width}" radius="${wheel_radius}"/>
+      </geometry>
+      <mass value="${wheel_mass}" />
+      <!-- According to https://en.wikipedia.org/wiki/List_of_moments_of_inertia#List_of_3D_inertia_tensors
+      We want Ixx = (1/12) * m * (3*r^2 + h^2) = 0.002374912 * (3 * 0.0345^2 + 0.018^2) = 0.00000925 = 9.25e-06
+              Iyy = (1/12) * m * (3*r^2 + h^2) = 0.002374912 * (3 * 0.0345^2 + 0.018^2) = 0.00000925 = 9.25e-06
+              Izz = (1/2) * m * r^2 = 0.01424947 * 0.0345^2 = 0.00001696 = 1.696e-05
+              -->
+      <inertia ixx="${(1/12) * wheel_mass * (3 * wheel_radius**2 + wheel_width**2)}" ixy="0" ixz="0"
+               iyy="${(1/12) * wheel_mass * (3 * wheel_radius**2 + wheel_width**2)}" iyz="0"
+               izz="${(1/2) * wheel_mass * wheel_radius**2}" />
       </inertial>
   </link>
@@ -62,5 +86,5 @@
     <parent link="base_link"/>
     <child link="wheel_right_link"/>
-    <origin xyz="0.0 -0.07 0.0345" rpy="0 0 0"/>
+    <origin xyz="0.0 -0.07 ${wheel_radius}" rpy="0 0 0"/>
     <axis xyz="0 1 0"/>
   </joint>
@@ -76,13 +100,18 @@
       <origin xyz="0 0 0" rpy="1.57 0 0"/>
       <geometry>
-        <cylinder length="0.018" radius="0.033"/>
+        <cylinder length="${wheel_width}" radius="${wheel_radius}"/>
       </geometry>
     </collision>
     <inertial>
-      <origin xyz="0 0 0" />
-      <mass value="2.8498940e-02" />
-      <inertia ixx="1.1175580e-05" ixy="-4.2369783e-11" ixz="-5.9381719e-09"
-               iyy="1.1192413e-05" iyz="-1.4400107e-11"
-               izz="2.0712558e-05" />
+      <origin xyz="0 0 0" rpy="1.57 0 0"/>
+      <mass value="${wheel_mass}" />
+      <!-- According to https://en.wikipedia.org/wiki/List_of_moments_of_inertia#List_of_3D_inertia_tensors
+      We want Ixx = (1/12) * m * (3*r^2 + h^2) = 0.002374912 * (3 * 0.0345^2 + 0.018^2) = 0.00000925 = 9.25e-06
+              Iyy = (1/12) * m * (3*r^2 + h^2) = 0.002374912 * (3 * 0.0345^2 + 0.018^2) = 0.00000925 = 9.25e-06
+              Izz = (1/2) * m * r^2 = 0.01424947 * 0.0345^2 = 0.00001696 = 1.696e-05
+              -->
+      <inertia ixx="${(1/12) * wheel_mass * (3 * wheel_radius**2 + wheel_width**2)}" ixy="0" ixz="0"
+               iyy="${(1/12) * wheel_mass * (3 * wheel_radius**2 + wheel_width**2)}" iyz="0"
+               izz="${(1/2) * wheel_mass * wheel_radius**2}" />
       </inertial>
   </link>
@@ -101,15 +130,20 @@
     </visual>
     <collision>
-      <origin xyz="0 0.0 0.005" rpy="0 0 0"/>
+      <origin xyz="0.0 -0.045 0.005" rpy="0 0 0"/>
       <geometry>
-        <box size="0.030 0.02 0.01"/>
+        <box size="${caster_colision_l} ${caster_colision_w} ${caster_colision_h}"/>
       </geometry>
     </collision>
     <inertial>
       <origin xyz="0 0 0" />
-      <mass value="0.005" />
-      <inertia ixx="0.001" ixy="0.0" ixz="0.0"
-               iyy="0.001" iyz="0.0"
-               izz="0.001" />
+      <mass value="${caster_mass}" />
+      <!-- According to https://en.wikipedia.org/wiki/List_of_moments_of_inertia#List_of_3D_inertia_tensors
+      We want Ixx = (1/12) * m * (h^2 + l^2) = 0.000041667 * (0.01^2 + 0.01^2) = 0.000000008 = 8e-09
+              Iyy = (1/12) * m * (w^2 + l^2) = 0.000041667 * (0.01^2 + 0.01^2) = 0.000000008 = 8e-09
+              Izz = (1/12) * m * (w^2 + h^2) = 0.000041667 * (0.01^2 + 0.01^2) = 0.000000008 = 8e-09
+              -->
+      <inertia ixx="${(1/12) * caster_mass * (caster_colision_l**2 + caster_colision_h**2)}" ixy="0" ixz="0"
+               iyy="${(1/12) * caster_mass * (caster_colision_w**2 + caster_colision_h**2)}" iyz="0"
+               izz="${(1/12) * caster_mass * (caster_colision_w**2 + caster_colision_l**2)}" />
     </inertial>
   </link>
