Commit message: Two sid wheels seem to be in place now.

File: ros/src/faricks_robot/urdf/farick.urdf.xacro (robot description, xacro)
@@ -8,10 +8,6 @@
   <xacro:property name="base_link_colision_h" value="0.01" />
   <xacro:property name="wheel_mass" value="0.160" />
-  <xacro:property name="wheel_width" value="0.04" />
+  <xacro:property name="wheel_width" value="0.06" />
   <xacro:property name="wheel_radius" value="0.06" />
-  <xacro:property name="caster_mass" value="0.0005" />
-  <xacro:property name="caster_colision_l" value="0.01" />
-  <xacro:property name="caster_colision_w" value="0.01" />
-  <xacro:property name="caster_colision_h" value="0.01" />
   <xacro:property name="stl_scale" value="0.001" />
   <link name="base_footprint"/>
@@ -19,9 +15,9 @@
     <parent link="base_footprint"/>
     <child link="base_link"/>
-    <origin xyz="0.0 0.0 0.00" rpy="0 0 0"/>
+    <origin xyz="0.0 0.0 0.0" rpy="0 0 0"/>
   </joint>
   <link name="base_link">
     <visual>
-      <origin xyz="0.0 0.0 0.0" rpy="0 0 3.14"/>
+      <origin xyz="0.242 -0.0765 -0.25" rpy="0 0 ${pi / 2}"/>
       <geometry>
         <mesh filename="package://faricks_robot/meshes/bottom_assembly.stl" scale="${stl_scale} ${stl_scale} ${stl_scale}"/>
@@ -30,5 +26,5 @@
     </visual>
     <collision>
-      <origin xyz="0.0 0.0 0.0315" rpy="0 0 0"/>
+      <origin xyz="0.0 0.0 0.0" rpy="0 0 0"/>
       <geometry>
         <box size="${base_link_colision_l} ${base_link_colision_w} ${base_link_colision_h}"/>
@@ -51,10 +47,9 @@
     <parent link="base_link"/>
     <child link="wheel_left_link"/>
-    <origin xyz="0.0 0.07 ${wheel_radius}" rpy="0 0 0"/>
-    <axis xyz="0 1 0"/>
+    <origin xyz="${base_link_colision_l / 2.0 - wheel_radius} ${base_link_colision_w / 2.0 - 0.025} ${-wheel_radius * 2}" rpy="0 0 0" />
   </joint>
   <link name="wheel_left_link">
     <visual>
-      <origin xyz="0 0.0 0.0" rpy="3.14 0 0"/>
+      <origin xyz="-0.0275 0.1075 -0.073" rpy="${pi / 2} 0 0"/>
       <geometry>
         <mesh filename="package://faricks_robot/meshes/wheel.stl" scale="${stl_scale} ${stl_scale} ${stl_scale}"/>
@@ -87,10 +82,9 @@
     <parent link="base_link"/>
     <child link="wheel_right_link"/>
-    <origin xyz="0.0 -0.07 ${wheel_radius}" rpy="0 0 0"/>
-    <axis xyz="0 1 0"/>
+    <origin xyz="${base_link_colision_l / 2.0 - wheel_radius} ${-base_link_colision_w / 2.0 + 0.025} ${-wheel_radius * 2}" rpy="0 0 0"/>
   </joint>
   <link name="wheel_right_link">
     <visual>
-      <origin xyz="0 0 0" rpy="0 0 0"/>
+      <origin xyz="-0.0275 -0.1075 0.073" rpy="${-pi / 2} 0 0"/>
       <geometry>
         <mesh filename="package://faricks_robot/meshes/wheel.stl" scale="${stl_scale} ${stl_scale} ${stl_scale}"/>
@@ -120,5 +114,5 @@
     <parent link="base_link"/>
     <child link="wheel_third_link"/>
-    <origin xyz="-0.0441 0.0435 0.0" rpy="0 0 0"/>
+    <origin xyz="${-base_link_colision_l / 2.0 - wheel_radius} 0 ${-wheel_radius * 2}" rpy="0 0 0"/>
   </joint>
   <link name="wheel_third_link">

Commit message: 3rd wheel is in place too now.

File: ros/src/faricks_robot/urdf/farick.urdf.xacro (robot description, xacro)
@@ -118,5 +118,5 @@
   <link name="wheel_third_link">
     <visual>
-      <origin xyz="0 0 0" rpy="0 0 0"/>
+      <origin xyz="-0.0275 -0.1075 0.073" rpy="${-pi / 2} 0 0"/>
       <geometry>
         <mesh filename="package://faricks_robot/meshes/wheel.stl" scale="${stl_scale} ${stl_scale} ${stl_scale}"/>

Commit message: Added the axis element to the wheel joints so that the wheels actually spin.

File: ros/src/faricks_robot/urdf/farick.urdf.xacro (robot description, xacro)
@@ -48,4 +48,5 @@
     <child link="wheel_left_link"/>
     <origin xyz="${base_link_colision_l / 2.0 - wheel_radius} ${base_link_colision_w / 2.0 - 0.025} ${-wheel_radius * 2}" rpy="0 0 0" />
+    <axis xyz="0 1 0"/>
   </joint>
   <link name="wheel_left_link">
@@ -83,4 +84,5 @@
     <child link="wheel_right_link"/>
     <origin xyz="${base_link_colision_l / 2.0 - wheel_radius} ${-base_link_colision_w / 2.0 + 0.025} ${-wheel_radius * 2}" rpy="0 0 0"/>
+    <axis xyz="0 1 0"/>
   </joint>
   <link name="wheel_right_link">
@@ -111,8 +113,9 @@
       </inertial>
   </link>
-  <joint name="wheel_third_joint" type="fixed">
+  <joint name="wheel_third_joint" type="continuous">
     <parent link="base_link"/>
     <child link="wheel_third_link"/>
     <origin xyz="${-base_link_colision_l / 2.0 - wheel_radius} 0 ${-wheel_radius * 2}" rpy="0 0 0"/>
+    <axis xyz="0 1 0"/>
   </joint>
   <link name="wheel_third_link">
